File: kicad/esp32_ym2149/_autosave-esp32_ym2149.kicad_pcb (KiCad board)
At the start: 2 copper layers, 26 parts, among them IC1 LM386, J1 5V_OUT, J2 3V3_OUT, U1 LM1086-5, U2 LM1086-3.3

Commit message: pcb draft extended
Parts:
- moved C5 25.4 mm to (162.6, 77.5)
- moved MCU1 25.4 mm to (182.9, 59.7)
- moved C1 5.24 mm to (111.8, 43.2)
- moved RV1 5.24 mm to (114.3, 36.8)
- moved IC1 5.24 mm to (123.2, 29.2)
- moved C2 5.08 mm to (128.3, 22.9)
- moved LS1 5.08 mm to (146.1, 33.0)
- moved C3 5.08 mm to (137.2, 40.6)
- moved C4 5.08 mm to (137.2, 30.5)
- moved C9 2.62 mm to (176.5, 87.6)
- moved C12 2.54 mm to (147.3, 96.5)
- moved C13 2.54 mm to (147.3, 87.6)
- moved C8 2.54 mm to (176.5, 96.5)
- moved C14 1.27 mm to (137.2, 49.5)
- moved POWER-SUPPLY1 1.27 mm to (208.3, 88.9)
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Routing:
- net AUDIO_CH_A: track 2.54 -> 43.1 mm
- net GNDREF: track 1.10 -> 29.2 mm
- net Net-(C3-Pad2): track 0.00 -> 9.96 mm
- net +5V: track 0.00 -> 8.98 mm
- net Net-(C3-Pad1): track 0.00 -> 8.67 mm
- net Net-(C2-Pad2): track 0.00 -> 7.63 mm
- net Net-(C2-Pad1): track 0.00 -> 7.40 mm
- net Net-(C1-Pad2): track 0.00 -> 5.20 mm
Changed lines of the file:
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@@
     (thickness 1.6)
     (drawings 0)
-    (tracks 2)
+    (tracks 29)
     (zones 0)
     (modules 26)
@@
   )
   (setup
-    (last_trace_width 0.25)
+    (last_trace_width 1)
+    (user_trace_width 1)
     (trace_clearance 0.2)
     (zone_clearance 0.508)
@@
   )
   (module Capacitor_THT:CP_Radial_D4.0mm_P2.00mm (layer F.Cu)
-    (at 106.68 44.45 90)
+    (at 111.76 43.18 90)
     (descr "CP, Radial series, Radial, pin pitch=2.00mm, , diameter=4mm, Electrolytic Capacitor")
     (tags "CP Radial series Radial pin pitch 2.00mm  diameter 4mm Electrolytic Capacitor")
@@
   )
   (module Capacitor_THT:CP_Radial_D4.0mm_P2.00mm (layer F.Cu)
-    (at 123.19 22.86 180)
+    (at 128.27 22.86 180)
     (descr "CP, Radial series, Radial, pin pitch=2.00mm, , diameter=4mm, Electrolytic Capacitor")
     (tags "CP Radial series Radial pin pitch 2.00mm  diameter 4mm Electrolytic Capacitor")
@@
   )
   (module Capacitor_THT:CP_Radial_D5.0mm_P2.50mm (layer F.Cu)
-    (at 132.08 40.64 90)
+    (at 137.16 40.64 90)
     (descr "CP, Radial series, Radial, pin pitch=2.50mm, , diameter=5mm, Electrolytic Capacitor")
     (tags "CP Radial series Radial pin pitch 2.50mm  diameter 5mm Electrolytic Capacitor")
@@
   )
   (module Capacitor_THT:CP_Radial_D5.0mm_P2.50mm (layer F.Cu)
-    (at 132.08 30.48 90)
+    (at 137.16 30.48 90)
     (descr "CP, Radial series, Radial, pin pitch=2.50mm, , diameter=5mm, Electrolytic Capacitor")
     (tags "CP Radial series Radial pin pitch 2.50mm  diameter 5mm Electrolytic Capacitor")
@@
   )
   (module Capacitor_THT:C_Rect_L4.6mm_W3.0mm_P2.50mm_MKS02_FKP02 (layer F.Cu)
-    (at 161.29 52.07 180)
+    (at 162.56 77.47 180)
     (descr "C, Rect series, Radial, pin pitch=2.50mm, , length*width=4.6*3.0mm^2, Capacitor, http://www.wima.de/DE/WIMA_MKS_02.pdf")
     (tags "C Rect series Radial pin pitch 2.50mm  length 4.6mm width 3.0mm Capacitor")
@@
   )
   (module Capacitor_THT:CP_Radial_D5.0mm_P2.00mm (layer F.Cu)
-    (at 184.15 93.98 90)
+    (at 184.15 95.25 90)
     (descr "CP, Radial series, Radial, pin pitch=2.00mm, , diameter=5mm, Electrolytic Capacitor")
     (tags "CP Radial series Radial pin pitch 2.00mm  diameter 5mm Electrolytic Capacitor")
@@
   )
   (module Capacitor_THT:CP_Radial_D5.0mm_P2.00mm (layer F.Cu)
-    (at 184.15 85.09 90)
+    (at 184.15 86.36 90)
     (descr "CP, Radial series, Radial, pin pitch=2.00mm, , diameter=5mm, Electrolytic Capacitor")
     (tags "CP Radial series Radial pin pitch 2.00mm  diameter 5mm Electrolytic Capacitor")
@@
   )
   (module Capacitor_THT:C_Disc_D4.3mm_W1.9mm_P5.00mm (layer F.Cu)
-    (at 176.53 93.98 90)
+    (at 176.53 96.52 90)
     (descr "C, Disc series, Radial, pin pitch=5.00mm, , diameter*width=4.3*1.9mm^2, Capacitor, http://www.vishay.com/docs/45233/krseries.pdf")
     (tags "C Disc series Radial pin pitch 5.00mm  diameter 4.3mm width 1.9mm Capacitor")
@@
   )
   (module Capacitor_THT:C_Disc_D4.3mm_W1.9mm_P5.00mm (layer F.Cu)
-    (at 176.53 85.01 90)
+    (at 176.53 87.63 90)
     (descr "C, Disc series, Radial, pin pitch=5.00mm, , diameter*width=4.3*1.9mm^2, Capacitor, http://www.vishay.com/docs/45233/krseries.pdf")
     (tags "C Disc series Radial pin pitch 5.00mm  diameter 4.3mm width 1.9mm Capacitor")
@@
   )
   (module Capacitor_THT:CP_Radial_D5.0mm_P2.00mm (layer F.Cu)
-    (at 156.21 93.98 90)
+    (at 156.21 95.25 90)
     (descr "CP, Radial series, Radial, pin pitch=2.00mm, , diameter=5mm, Electrolytic Capacitor")
     (tags "CP Radial series Radial pin pitch 2.00mm  diameter 5mm Electrolytic Capacitor")
@@
   )
   (module Capacitor_THT:CP_Radial_D5.0mm_P2.00mm (layer F.Cu)
-    (at 156.21 85.09 90)
+    (at 156.21 86.36 90)
     (descr "CP, Radial series, Radial, pin pitch=2.00mm, , diameter=5mm, Electrolytic Capacitor")
     (tags "CP Radial series Radial pin pitch 2.00mm  diameter 5mm Electrolytic Capacitor")
@@
   )
   (module Capacitor_THT:C_Disc_D4.3mm_W1.9mm_P5.00mm (layer F.Cu)
-    (at 147.32 93.98 90)
+    (at 147.32 96.52 90)
     (descr "C, Disc series, Radial, pin pitch=5.00mm, , diameter*width=4.3*1.9mm^2, Capacitor, http://www.vishay.com/docs/45233/krseries.pdf")
     (tags "C Disc series Radial pin pitch 5.00mm  diameter 4.3mm width 1.9mm Capacitor")
@@
   )
   (module Capacitor_THT:C_Disc_D4.3mm_W1.9mm_P5.00mm (layer F.Cu)
-    (at 147.32 85.09 90)
+    (at 147.32 87.63 90)
     (descr "C, Disc series, Radial, pin pitch=5.00mm, , diameter*width=4.3*1.9mm^2, Capacitor, http://www.vishay.com/docs/45233/krseries.pdf")
     (tags "C Disc series Radial pin pitch 5.00mm  diameter 4.3mm width 1.9mm Capacitor")
@@
   )
   (module Capacitor_THT:C_Rect_L4.6mm_W3.0mm_P2.50mm_MKS02_FKP02 (layer F.Cu)
-    (at 138.43 49.53 270)
+    (at 137.16 49.53 270)
     (descr "C, Rect series, Radial, pin pitch=2.50mm, , length*width=4.6*3.0mm^2, Capacitor, http://www.wima.de/DE/WIMA_MKS_02.pdf")
     (tags "C Rect series Radial pin pitch 2.50mm  length 4.6mm width 3.0mm Capacitor")
@@
   )
   (module Package_DIP:DIP-8_W7.62mm_Socket (layer F.Cu)
-    (at 118.11 30.48)
+    (at 123.19 29.21)
     (descr "8-lead though-hole mounted DIP package, row spacing 7.62 mm (300 mils), Socket")
     (tags "THT DIP DIL PDIP 2.54mm 7.62mm 300mil Socket")
@@
   )
   (module Connector_PinHeader_2.54mm:PinHeader_2x01_P2.54mm_Vertical (layer F.Cu)
-    (at 139.7 93.98 90)
+    (at 139.7 95.25 90)
     (descr "Through hole straight pin header, 2x01, 2.54mm pitch, double rows")
     (tags "Through hole pin header THT 2x01 2.54mm double row")
@@
   )
   (module Connector_PinHeader_2.54mm:PinHeader_2x01_P2.54mm_Vertical (layer F.Cu)
-    (at 139.7 85.09 90)
+    (at 139.7 86.36 90)
     (descr "Through hole straight pin header, 2x01, 2.54mm pitch, double rows")
     (tags "Through hole pin header THT 2x01 2.54mm double row")
@@
   )
   (module Connector_PinSocket_2.54mm:PinSocket_2x01_P2.54mm_Vertical (layer F.Cu)
-    (at 140.97 33.02 90)
+    (at 146.05 33.02 90)
     (descr "Through hole straight socket strip, 2x01, 2.54mm pitch, double cols (from Kicad 4.0.7), script generated")
     (tags "Through hole socket strip THT 2x01 2.54mm double row")
@@
   )
   (module MODULE_ESP32-DEVKITC-32D (layer F.Cu)
-    (at 181.61 34.29 90)
+    (at 182.88 59.69 90)
     (fp_text reference MCU1 (at -10.829175 -28.446045 90) (layer F.SilkS)
       (effects (font (size 1.000386 1.000386) (thickness 0.015)))
@@
   )
   (module Connector_PinSocket_2.54mm:PinSocket_2x01_P2.54mm_Vertical (layer F.Cu)
-    (at 208.28 87.63 90)
+    (at 208.28 88.9 90)
     (descr "Through hole straight socket strip, 2x01, 2.54mm pitch, double cols (from Kicad 4.0.7), script generated")
     (tags "Through hole socket strip THT 2x01 2.54mm double row")
@@
   )
   (module Potentiometer_THT:Potentiometer_Vishay_148-149_Single_Vertical (layer F.Cu)
-    (at 109.22 38.1 90)
+    (at 114.3 36.83 90)
     (descr "Potentiometer, vertical, Vishay 148-149 Single, http://www.vishay.com/docs/57040/148149.pdf")
     (tags "Potentiometer vertical Vishay 148-149 Single")
@@
   )
   (module Package_DIP:DIP-40_W25.4mm (layer F.Cu)
-    (at 106.68 49.53)
+    (at 106.68 48.26)
     (descr "40-lead though-hole mounted DIP package, row spacing 25.4 mm (1000 mils)")
     (tags "THT DIP DIL PDIP 2.54mm 25.4mm 1000mil")
@@
     )
   )
-  (segment (start 106.68 54.61) (end 106.68 57.15) (width 0.25) (layer F.Cu) (net 2))
-  (segment (start 140.97 31.92) (end 140.97 33.02) (width 0.25) (layer F.Cu) (net 7))
+  (segment (start 111.76 41.18) (end 110.911472 41.18) (width 0.25) (layer F.Cu) (net 1))
+  (segment (start 111.76 36.83) (end 111.76 41.18) (width 1) (layer F.Cu) (net 1))
+  (segment (start 105.179999 51.839999) (end 105.880001 52.540001) (width 1) (layer F.Cu) (net 2))
+  (segment (start 105.880001 52.540001) (end 106.68 53.34) (width 1) (layer F.Cu) (net 2))
+  (segment (start 108.899998 43.18) (end 105.179999 46.899999) (width 1) (layer F.Cu) (net 2))
+  (segment (start 105.179999 46.899999) (end 105.179999 51.839999) (width 1) (layer F.Cu) (net 2))
+  (segment (start 111.76 43.18) (end 108.899998 43.18) (width 1) (layer F.Cu) (net 2))
+  (segment (start 132.08 53.34) (end 106.68 53.34) (width 1) (layer F.Cu) (net 2))
+  (segment (start 106.68 55.88) (end 106.68 53.34) (width 1) (layer F.Cu) (net 2))
+  (segment (start 130.81 25.4) (end 128.27 22.86) (width 1) (layer F.Cu) (net 3))
+  (segment (start 130.81 29.21) (end 130.81 25.4) (width 1) (layer F.Cu) (net 3))
+  (segment (start 123.19 25.94) (end 126.27 22.86) (width 1) (layer F.Cu) (net 4))
+  (segment (start 123.19 29.21) (end 123.19 25.94) (width 1) (layer F.Cu) (net 4))
+  (segment (start 130.81 36.83) (end 130.81 38.1) (width 1) (layer F.Cu) (net 5))
+  (segment (start 133.35 40.64) (end 137.16 40.64) (width 1) (layer F.Cu) (net 5))
+  (segment (start 130.81 38.1) (end 133.35 40.64) (width 1) (layer F.Cu) (net 5))
+  (segment (start 143.47 38.14) (end 146.05 35.56) (width 1) (layer F.Cu) (net 6))
+  (segment (start 137.16 38.14) (end 143.47 38.14) (width 1) (layer F.Cu) (net 6))
+  (segment (start 146.05 31.92) (end 146.05 33.02) (width 0.25) (layer F.Cu) (net 7))
+  (segment (start 146.05 31.17) (end 146.05 33.02) (width 1) (layer F.Cu) (net 7))
+  (segment (start 142.86 27.98) (end 146.05 31.17) (width 1) (layer F.Cu) (net 7))
+  (segment (start 137.16 27.98) (end 142.86 27.98) (width 1) (layer F.Cu) (net 7))
+  (segment (start 114.3 38.102792) (end 114.3 36.83) (width 1) (layer F.Cu) (net 7))
+  (segment (start 114.3 43.100002) (end 114.3 38.102792) (width 1) (layer F.Cu) (net 7))
+  (segment (start 109.140002 48.26) (end 114.3 43.100002) (width 1) (layer F.Cu) (net 7))
+  (segment (start 106.68 48.26) (end 109.140002 48.26) (width 1) (layer F.Cu) (net 7))
+  (segment (start 137.16 32.28) (end 135.15 34.29) (width 1) (layer F.Cu) (net 8))
+  (segment (start 137.16 30.48) (end 137.16 32.28) (width 1) (layer F.Cu) (net 8))
+  (segment (start 135.15 34.29) (end 130.81 34.29) (width 1) (layer F.Cu) (net 8))
 )
